File: labs_soluzioni/lab4/lab4.kicad_sch (KiCad schematic)
At the start: 1 part, among them U1 XC7A35T-FGG484

Commit message: NEW lab4
Parts:
- removed U1: XC7A35T-FGG484, Package_BGA:BGA484C100P22X22_2300X2300X260, symbol FPGA_Xilinx_Artix7:XC7A35T-FGG484
Other:
- removed sheet gtr
- removed sheet io1
- removed sheet io2
- removed sheet io3
- added sheet FTDI2232H (ftdi.kicad_sch)
- added sheet GPIOS (gpios.kicad_sch)
- added sheet POWER (power.kicad_sch)
- added sheet RAM (ram.kicad_sch)
- added sheet SPARTAN6 (spartan6.kicad_sch)
- note added: "CSG324"
- note added: "FT2232H"
- note added: "GPIOs"
- note added: "LPDDR"
- note added: "POWER SUPPLY"
- note added: "SPARTAN 6 FPGA"
- company: (none) -> Numato Lab
- title: (none) -> SATURN SPARTAN6 FPGA MODULE
